File: parts/arm/encoder/encoder_nano_adapter/encoder_nano_adapter.kicad_pcb (KiCad board)
At the start: 2 copper layers, 48.2 x 24.1 mm, 4 parts, among them J1 AS5600_power, J2 AS5600_I2C, J3 Servo

Commit message: Stretch the wiretube so you can feed a USB or Anderson through while assembled.  Also added mounting screw to nano adapter board.
Connections:
- A1 pad 27: Net-(A1-+5V) -> unconnected-(A1-+5V-Pad27)
- J3 pad 2: Net-(A1-+5V) -> unconnected-(J3-Pin_2-Pad2)
Routing:
- net Net-(A1-+5V): track 20.8 -> 0.00 mm
- net Net-(J3-Pin_1): track 21.7 -> 15.8 mm
Other:
- board size 48.2 x 24.1 mm -> 48.2 x 22 mm
